Commit message: debug: mitigate robot lurch when braking
Changed odometrySource parameter in robot description to 'encoder' so gmapping zero is at robot initial pose, different from Gazebo zero. This makes it so that map built by either turtlebot or ryabot can be used by both.

File: ryabot/urdf/ryabot.xacro (robot description, xacro)
@@ -8,10 +8,10 @@
         <pose>0 0 0.05 0 0 0</pose>
         <inertial>
-            <mass value="5.0" />
-            <origin xyz="0 0 0" rpy="0 0 0" />
-            <inertia
-                ixx="0.1" ixy="0" ixz="0"
-                iyy="0.1" iyz="0"
-                izz="0.1"
+            <mass value="7.50" />
+            <origin xyz="0 0 0" rpy="0 0 0" />
+            <inertia
+                ixx="0.2" ixy="0" ixz="0"
+                iyy="0.2" iyz="0"
+                izz="0.2"
             />
         </inertial>

Commit message: debug: tune planner/amcl parameters
Not successful yet, but checkpoint.

File: ryabot/urdf/ryabot.xacro (robot description, xacro)
@@ -4,14 +4,14 @@
     <xacro:include filename="$(find ryabot)/urdf/ryabot.gazebo" />
     <!-- define robot links -->
-    <link name="robot_footprint"></link>
+    <link name="base_footprint"></link>
     <link name="chassis">
         <pose>0 0 0.05 0 0 0</pose>
         <inertial>
-            <mass value="7.50" />
-            <origin xyz="0 0 0" rpy="0 0 0" />
-            <inertia
-                ixx="0.2" ixy="0" ixz="0"
-                iyy="0.2" iyz="0"
-                izz="0.2"
+            <mass value="5.00" />
+            <origin xyz="0 0 0" rpy="0 0 0" />
+            <inertia
+                ixx="0.1" ixy="0" ixz="0"
+                iyy="0.1" iyz="0"
+                izz="0.01"
             />
         </inertial>
@@ -184,5 +184,5 @@
     <joint name="robot_footprint_joint" type="fixed">
         <origin xyz="0 0 0" rpy="0 0 0" />
-        <parent link="robot_footprint" />
+        <parent link="base_footprint" />
         <child link="chassis" />
     </joint>
